File: power.kicad_sch (KiCad schematic)
At the start: 38 parts, among them J10 Conn_01x02, J14 Conn_01x02, J25 Conn_01x02, J26 Conn_01x02, J9 Conn_01x02, Q1 2N7002, U1 AP2112K-3.3, U12 Ag9905LP

Commit message: changed 24V connector
Parts:
- J10: footprint easyeda2kicad:CONN-TH_P5.00_KF243-5.0-2P -> easyeda2kicad:CONN-TH_4P-P5.00_1862411
Changed lines of the file:
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@@
 			)
 		)
-		(property "Footprint" "easyeda2kicad:CONN-TH_P5.00_KF243-5.0-2P"
+		(property "Footprint" "easyeda2kicad:CONN-TH_4P-P5.00_1862411"
 			(at 179.07 40.64 0)
 			(effects
