File: i2c.kicad_sch (KiCad schematic)
At the start: 23 parts, among them IC3 MTCH112-I_SN, J13 Conn_01x02, J15 Conn_01x04, U4 TMP112xxDRL, U9 TMP112xxDRL

Commit message: updated LED resistor values
Other:
- moved on the sheet: C13, C41, J15, JP10, JP11, JP12, JP13, JP6, JP7, JP8, JP9, R41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
