File: led.kicad_sch (KiCad schematic)
At the start: 7 parts, among them J1 Conn_01x22, J17 Conn_01x22

Commit message: updated LED resistor values
Parts:
- R1, R73: value 680R -> 1k; LCSC C23228 -> C21190
Changed lines of the file:
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@@
 			)
 		)
-		(property "Value" "680R"
+		(property "Value" "1k"
 			(at 149.9432 46.99 90)
 			(effects
@@
 			)
 		)
-		(property "LCSC" "C23228"
+		(property "LCSC" "C21190"
 			(at 152.4 46.99 0)
 			(effects
@@
 			)
 		)
-		(property "Value" "680R"
+		(property "Value" "1k"
 			(at 149.9432 81.28 90)
 			(effects
@@
 			)
 		)
-		(property "LCSC" "C23228"
+		(property "LCSC" "C21190"
 			(at 152.4 81.28 0)
 			(effects
