File: config.kicad_sch (KiCad schematic)
At the start: 47 parts, among them Q4 2N7002, SW3 SW_SPDT

Commit message: updated LED resistor values
Parts:
- D14: value LED_24V -> LED_24V_FUSED; LCSC C2297 -> C34499; color green -> white
- D36: value LED_5V_EXT -> LED_5V_PoE
- D37: value LED_5V_EXT -> LED_5V_USB
- D38: value LED_5V_FUSED -> LED_5V_CONN; LCSC C34499 -> C2297; color white -> green
- D39: value LED_5V_FUSED -> LED_5V_FUSED_IN; LCSC C34499 -> C2297; color white -> green
- R18: value 1k -> 10k; LCSC C21190 -> C25804
- R19: value 1k -> 47k; LCSC C21190 -> C25819
- R26, R76, R87, R88, R90, R91: value 1k -> 4.7k; LCSC C21190 -> C23162
Other:
- moved on the sheet: D13, D15, D23, R18, R19, R26, R77

Commit message: schematic annotation
Other:
- moved on the sheet: D13, D14, D36, D37, D38, D39, Q4, R18, R19, R87, R88, R90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
